Commit message: 複数のロボットをシミュレーションするためのlaunchファイルを更新し、robot.urdfに物理特性を追加。必要な依存関係をpackage.xmlに追加。

File: src/inrof_sim/urdf/robot.urdf (robot description, URDF)
Before this commit: robot robot, 2 links, 1 joints
Links:
- link base_link: mass None -> 1.0; geometry collision box size=0.1 0.1 0.1; visual box size=0.1 0.1 0.1
