Commit message: robot.urdfのリンク名を修正し、Gazeboプラグインの名前を更新。システムの整合性を向上させるために、親リンクをbase_footprintに変更。
Co-authored-by: Copilot <copilot@github.com>

File: src/inrof_sim/urdf/robot.urdf (robot description, URDF)
Before this commit: robot robot, 2 links, 1 joints
Links:
- removed link base_root
- added link base_footprint
Joints:
- joint body_joint: parent base_root -> base_footprint
